File: KiCad/Breadboard8088PCV2/BBPCV2PLDS.kicad_sch (KiCad schematic)
At the start: 27 parts, among them U100 74HC74, U101 74LS04, U102 74LS07, U103 74LS08, U104 74HC74, U105 74HC74, U106 74LS07, U39 74LS08, U42 74LS04, U45 74LS00, U5 74LS08, U6 74LS08, U7 74LS04, U8 74LS32, U88 74LS04, U89 74HC74, U90 74LS00, U91 74LS74, U92 74LS74, U93 74LS08, U94 74LS32, U95 74LS32, U96 74LS32, U97 74LS32, U98 74HC74, U99 74LS32

Commit message: Updates as of Video 14
CGA PLD files and updated KiCad schematic as of video 14 of BBPCV2
Parts:
- added U10, U21: 74LS574BB, symbol Breadboarding:74LS574BB
- added U107: ATF16V8B_BLINKSYNC, symbol Breadboarding:GAL16V8BB
- added U108, U109: ATF22V10C, symbol Breadboarding:ATF22LV10
- added U12: ATF22V10C_CGACOLMUX, symbol Breadboarding:ATF22LV10_VIDEO2
- added U13: ATF22V10C_VIDEOOUT, symbol Breadboarding:ATF22LV10_VIDEO2
- added U16: ATF22LV10_CGACLOCK, symbol Breadboarding:ATF22LV10_VIDEO2
- added U17: ATF22LV10, symbol Breadboarding:ATF22LV10
- added U18: 74LS174BB, symbol Breadboarding:74LS174BB
- added U20: 74LS74BB, symbol Breadboarding:74LS74BB
- added Y8: MXO45HS-3C-25M1750, symbol Breadboarding:MXO45HS-3C-25M1750
Connections:
- net ~{MEMR}: now also U108.11 (~{MEMR}), U109.10 (~{MEMR})
- net ~{RESET}: now also U13.11 (~{RESET}), U16.6 (~{RST}), U18.1 (~{Mr})
- new net: U10.20 (VCC), U107.20 (VCC), U12.24 (VCC), U13.24 (VCC), U16.24 (VCC), U17.24 (VCC), U18.16 (VCC), U20.1 (~{1CLR}), U20.10 (~{2PRE}), U20.13 (~{2CLR}), U20.14 (VCC), U20.4 (~{1PRE}), U21.20 (VCC), Y8.8 (VCC)
- new net: U107.10 (GND), U107.4 (InvVS), U109.12 (GND), U21.10 (GND)
- new net  ~{MEMW}: U109.9 (~{MEMW})
- new net +AlphaDots: U12.19 (+AlphaDots), U13.14 (+AlphaDots), U17.11 (+AlphaDots)
- new net +B/W: U18.7 (Q2)
- new net +En Blink: U13.8 (BlinkEn), U17.2 (+EnBlink), U18.15 (Q5)
- new net +VideoEnable: U13.5 (Video_En), U18.10 (Q3)
- new net 25Mhz: U16.1 (25Mhz), Y8.5 (OUTPUT)
- new net 640BW: U108.5 (640BW), U12.9 (640BW), U16.3 (640BW), U18.12 (Q4)
- new net AD0: U17.10 (AD0), U21.12 (Q0)
- new net AD1: U17.9 (AD1), U21.13 (Q1)
- new net AD2: U17.8 (AD2), U21.14 (Q2)
- new net AD3: U17.7 (AD3), U21.15 (Q3)
- new net AD4: U17.6 (AD4), U21.16 (Q4)
- new net AD5: U17.5 (AD5), U21.17 (Q5)
- new net AD6: U17.4 (AD6), U21.18 (Q6)
- new net AD7: U17.3 (AD7), U21.19 (Q7)
- new net ADCLK: U108.16 (ADCLK)
- new net AT7: U13.13 (AT7), U17.22 (AT7)
- new net ATSRLatch: U16.23 (ATSRLatch), U21.11 (CLK)
- new net B: U12.8 (B), U17.15 (B)
- new net Blank/~{DE}: U107.17 (Blank/~{DE}), U13.7 (Blank/~{DE})
- new net BlinkChr: U107.16 (BlkChrQ4), U13.3 (BlinkChr)
- new net BlinkCur: U107.15 (BlkCurQ3), U13.4 (BlinkCur)
- new net C0: U12.3 (C0), U17.20 (C0)
- new net C1: U12.4 (C1), U17.19 (C1)
- new net CAB: U108.21 (CAB)
- new net CHLatch: U16.20 (CHLatch)
- new net CPUACT: U109.19 (CPUACT), U20.12 (2D)
- new net CPUACTDCLK: U108.1 (CLK), U109.18 (CPUACTDCLK)
- new net CPUACTS1: U108.9 (CPUACTS1), U109.20 (CPUACTS1), U20.5 (1Q)
- new net CPUACTSYNC: U109.1 (CLK), U20.2 (1D), U20.9 (2Q)
- new net CQa: U107.5 (InvHS), U108.2 (CQa), U108.24 (VCC), U109.23 (CQa), U109.24 (VCC)
- new net CQb: U108.3 (CQb), U109.22 (CQb)
- new net CQc: U108.4 (CQc), U109.21 (CQc)
- new net CRBLue: U10.12 (Q0), U12.23 (CRblue)
- new net CRBackInten: U10.16 (Q4), U12.2 (CRBkInten)
- new net CRColourSel: U10.17 (Q5), U12.1 (CRColSel)
- new net CRGreen: U10.13 (Q1), U12.22 (CRGreen)
- new net CRIntensity: U10.15 (Q3), U12.13 (CRInten)
- new net CRRed: U10.14 (Q2), U12.21 (CRRed)
- new net Char Clk: U109.4 (Qc), U13.1 (Char_Clk), U16.17 (Qc), U17.14 (Qc)
- new net Cursor: U13.2 (Cursor)
- new net D0: U10.9 (D0), U18.3 (D0)
- new net D1: U10.8 (D1), U18.4 (D1)
- new net D2: U10.7 (D2), U18.6 (D2)
- new net D3: U10.6 (D3), U18.11 (D3)
- new net D4: U10.5 (D4), U18.13 (D4)
- new net D5: U10.4 (D5), U18.14 (D5)
- new net D6: U10.3 (D6)
- new net D7: U10.2 (D7)
- new net DE: U107.9 (DE)
- new net DIR: U108.8 (DIR), U109.17 (DIR)
- new net D[0..7]: U10.1 (~{OE}), U10.10 (GND), U107.11 (~{OE}), U108.12 (GND), U12.12 (GND), U13.12 (GND), U16.12 (GND), U17.12 (GND), U18.8 (GND), U20.7 (GND), U21.1 (~{OE}), Y8.4 (GND)
- new net DotClk: U109.6 (DotClk), U16.14 (DotClkBuf), U20.11 (2CLK), U20.3 (1CLK)
- new net G: U12.7 (G), U17.16 (G)
- new net GRPH: U108.7 (GRPH), U12.11 (GRPH), U16.13 (GRPH), U17.23 (GRPH), U18.5 (Q1)
- new net H Sync: U107.18 (HSout), U107.3 (HSin), U13.23 (HS)
- new net HIRES: U108.6 (HIRES), U16.2 (HIRES), U18.2 (Q0)
- new net HSync Dly: U13.21 (HSDly)
- new net I: U12.5 (I), U17.18 (I)
- new net Overscan: U12.18 (Overscan), U13.18 (Overscan)
- new net P0: U12.14 (P0)
- new net P1: U12.15 (P1)
- new net P2: U12.16 (P2)
- new net P3: U12.17 (P3)
- new net Qa: U109.2 (Qa), U16.19 (Qa)
- new net Qb: U109.3 (Qb), U16.18 (Qb), U17.13 (Qb)
- new net Qd: U109.5 (Qd), U16.22 (Qd)
- new net R: U12.6 (R), U17.17 (R)
- new net S Dots: U13.6 (S_Dots)
- new net V Sync: U107.1 (CLK), U107.19 (VSout), U107.2 (VSin), U13.22 (VS)
- new net VD0: U21.9 (D0)
- new net VD1: U21.8 (D1)
- new net VD2: U21.7 (D2)
- new net VD3: U21.6 (D3)
- new net VD4: U21.5 (D4)
- new net VD5: U21.4 (D5)
- new net VD6: U21.3 (D6)
- new net VD7: U21.2 (D7)
- new net VSync Dly: U13.20 (VSDly)
- new net ~{646OE}: U109.14 (~{646OE})
- new net ~{ADOE}: U108.19 (~{ADOE}), U109.8 (~{ADOE})
- new net ~{CBA}: U108.20 (~{CBA})
- new net ~{CGACOL}: U10.11 (CLK)
- new net ~{CGACONT}: U18.9 (Cp)
- new net ~{CGARAM}: U108.13 (~{CGARAM}), U109.11 (~{CGARAM})
- new net ~{CH}/AT: U16.21 (~{CH}/AT)
- new net ~{CLR_SR}: U13.15 (~{CLR_SR}), U17.21 (~{CLR_SR})
- new net ~{Char Clk}: U16.16 (~{Qc}ChrClk)
- new net ~{RDY}/WAIT: U108.17 (RDY/WAIT)
- new net ~{VAOE}: U109.15 (~{VAOE})
- new net ~{VROE}: U109.16 (~{VROE})
- new net ~{VRWE}: U108.18 (~{VRWE}), U109.7 (~{VRWE})
- no-connect marks 6 -> 38
Other:
- note added: "25.175MHz"
- note added: "Attribute Latch"
- note added: "Attribute Multiplexer PLD"
- note added: "Blink Divider and HS VS"
- note added: "CGA Colour Register"
- note added: "CGA Control Register"
- note added: "CGA Logic PLD 2"
- note added: "CGA VIDEO CONTROLLER"
- note added: "CRTC HD68A45S"
- note added: "Clock PLD"
- note added: "Colour Multiplexer PLD"
- note added: "First Flip Flop Syncs the CPUACT with the video Dot Clock so we don't have short DC Cycles from DCQ0-3"
- note added: "Inverted Display Enable high during blanking period for status reg."
- note added: "Note CRTC uses inverted Qc character clock, Qa and Qb are not inverted"
- note added: "Second Flip Flop delays the CPUACTSYNC by one video Dot Clock cycle otherwise we miss last Gated Dot Clock from CPUACTDCLK. CPUACTS1 ORed with CPUACTSYNC is used to gate the Dot Clock so it is extended."
- note added: "Shift Register"
- note added: "Video DAC"
- note added: "Video Output PLD"
