File: KiCad/Breadboard8088PCV2/Breadboard8088PCV2.kicad_sch (KiCad schematic)
At the start: 172 parts, among them IC1 MIC1232NY, J2 IDE/ATA Disk, J3 Floppy Disk 1-34, J4 Mini-DIN-6, J5 Mini-DIN-6, J6 Power On Self Test Port, J7 DB15_Female_HighDensity, Q1 PN2222A, SW1 S, SW10 ES, SW11 7, SW12 8, SW13 9, SW14 E, SW15 M, SW16 4, SW17 5, SW18 6, SW19 A, SW2 L, SW20 R, SW21 1, SW22 2, SW23 3, SW24 0, SW25 I, SW26 AB, SW27 RST, SW3 CN, SW4 G, SW5 CS, SW6 A, SW7 B, SW8 C, SW9 D, U1 Intersil 80C88 BB Layout, U11 ATF22V10C_IODECODE2, U19 USBFT232, U2 74LS646, U22 7_Segment_x_4_LED_Nanocomp_RH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, U23 ULN2803A, U24 ATF22V10C_IODECODE1, U26 7_Segment_x_4_LED_Nanocomp, U27 TL16C550D, U28 ATF22V10C, U29 74LS574BB_POST, U3 ATF16V8B, U30 28C256_BBPIN, U31 ASC6C4008_DIP32_BBPIN, U32 ATF22LV10, U34 8253, U35 ATF750C_RDYWSPKR, U36 74LS541BB_PORTBR, U37 74LS175_PORTBW, U38 WD37C65C, U4 74LS145, U40 VT82C42N, U41 74LS06, U44 DS12885, U46 74LS245, U47 74LS646, U48 ATF22LV10, U49 ATF750C, U50 ASC6C4008_DIP32_BBPIN, U51 74LS245, U52 74LS573B, U53 74LS573B, U54 74LS541BB, U55 74LS245, U56 8259A_PIC1, U57 8259A_PIC2, U58 ATF16V8B_BLINKSYNC, U59 ATF22V10C_CGACOLMUX, U60 ATF22V10C_VIDEOOUT, U61 LM334Z, U62 IMS176G, U63 ATF22LV10_CGACLOCK, U64 ATF22LV10, U65 74LS174BB, U66 28C64_BBPIN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

Commit message: Updates as of Video 14
CGA PLD files and updated KiCad schematic as of video 14 of BBPCV2
Parts:
- removed R56, R57, R58, R59, R60: 4k7, symbol Device:R
- removed unit 5 of U41
- removed U58: ATF16V8B_BLINKSYNC, symbol Breadboarding:GAL16V8BB
- removed U59: ATF22V10C_CGACOLMUX, symbol Breadboarding:ATF22LV10_VIDEO2
- removed U60: ATF22V10C_VIDEOOUT, symbol Breadboarding:ATF22LV10_VIDEO2
- removed U63: ATF22LV10_CGACLOCK, symbol Breadboarding:ATF22LV10_VIDEO2
- removed U64: ATF22LV10, symbol Breadboarding:ATF22LV10
- removed U65: 74LS174BB, symbol Breadboarding:74LS174BB
- removed U70: 74LS541B, symbol Breadboarding:74LS541BB
- removed U78, U83: 74LS574BB, symbol Breadboarding:74LS574BB
- removed U81, U84: ATF22V10C, symbol Breadboarding:ATF22LV10
- removed U82: ATF16V8B, symbol Breadboarding:ATF16V8BB
- removed U85: 74LS74BB, symbol Breadboarding:74LS74BB
- removed Y7: MXO45HS-3C-25M1750, symbol Breadboarding:MXO45HS-3C-25M1750
- added J1: ATMEL-JTAG-10, symbol Breadboarding:ATMEL-JTAG-10
- added R14, R16: 10K, symbol Device:R
- added U14: ATF1508AS7AU100, Package_QFP:TQFP-100_14x14mm_P0.5mm, symbol Breadboarding:ATF1504AS10AU100 On breadboard adapter 26 pins high x 24 pins wide
- added U15: ATF1504AS_44PIN_DIP, Package_DIP:DIP-44, symbol Breadboarding:ATF1504AS_44PIN_DIP
- added U9: 74LS06, symbol 74xx:74LS06
Connections:
- net DIR is gone; now on net DT/R: U73.3 (DIR)
- net DT/~{R} is gone; now on net DT/R: U1.27 (DT/~{R}), U3.5 (DT/~{R}), U55.1 (A->B), U86.18 (Y0), U86.2 (A0), U87.1 (A->B)
- net  ~{IOR}: now also U15.35 (~{IOR})
- net  ~{IOW}: now also U15.34 (~{IOW})
- net  ~{MEMW}: now also U15.25 (~{MEMW})
- net 13: no longer U68.39 (HS)
- net 14: no longer U68.40 (VS)
- net ADCLK: now also U15.30 (ADCLK)
- net ATSRLatch: now also U14.44 (ATSRLATCH)
- net CAB: now also U15.2 (CAB)
- net CHLatch: now also U14.40 (CHLATCH)
- net Cursor: now also U14.83 (CURSOR)
- net D0: now also U14.52 (DO)
- net D1: now also U14.54 (D1)
- net D2: now also U14.56 (D2)
- net D3: now also U14.58 (D3)
- net D4: now also U14.60 (D4)
- net D5: now also U14.64 (D5)
- net D6: now also U14.68 (D6)
- net D7: now also U14.70 (D7)
- net DE: now also U14.81 (DE)
- net DotClk: now also U14.93 (DOTCLK), U15.37 (GCLK1); no longer U67.7 (Clk)
- net E: now also U69.17 (E); no longer U69.16 (E)
- net GRPH: now also U14.46 (GRPH), U15.20 (GRPH)
- net HIRES: now also U14.47 (HIRES), U15.19 (HIRES)
- net ID0: now also U51.11 (B7); no longer U51.18 (B0)
- net ID1: now also U51.12 (B6); no longer U51.17 (B1)
- net ID10: now also U47.15 (B5); no longer U47.18 (B2)
- net ID11: now also U47.16 (B4); no longer U47.17 (B3)
- net ID12: now also U47.17 (B3); no longer U47.16 (B4)
- net ID13: now also U47.18 (B2); no longer U47.15 (B5)
- net ID14: now also U47.19 (B1); no longer U47.14 (B6)
- net ID15: now also U47.20 (B0); no longer U47.13 (B7)
- net ID2: now also U51.13 (B5); no longer U51.16 (B2)
- net ID3: now also U51.14 (B4); no longer U51.15 (B3)
- net ID4: now also U51.15 (B3); no longer U51.14 (B4)
- net ID5: now also U51.16 (B2); no longer U51.13 (B5)
- net ID6: now also U51.17 (B1); no longer U51.12 (B6)
- net ID7: now also U51.18 (B0); no longer U51.11 (B7)
- net ID8: now also U47.13 (B7); no longer U47.20 (B0)
- net ID9: now also U47.14 (B6); no longer U47.19 (B1)
- net Keyboard Clock: now also C4.1, J5.5, R12.1; no longer C6.2, C7.1, J4.1, J4.5, R10.1, R9.1, U40.27 (P10), U41.4
- net Mouse Clock: now also C7.1, J4.5, R10.1, U41.8; no longer C4.1, J5.5, R12.2
- net Mouse Data: now also C6.2, J4.1, R9.1, U9.10; no longer C5.1, J5.1, R11.2, U41.8
- net P0: now also U14.96 (P0)
- net P1: now also U14.97 (P1)
- net P2: now also U14.98 (P2)
- net P22: now also U9.11; no longer U41.9
- net P23: now also U41.9
- net P3: now also U14.99 (P3)
- net Qa: now also U14.20 (Qa), U15.10 (Qa)
- net Qb: now also U14.21 (Qb), U15.11 (Qb)
- net Qd: now also U14.25 (Qd), U15.13 (Qd)
- net S Dots: now also U14.42 (SDOTS)
- net VCC: now also R11.2, R12.2, R14.2, R16.2, U14.18 (VCC), U14.3 (VCC), U14.34 (VCC), U14.39 (VCCint), U14.51 (VCC), U14.66 (VCC), U14.82 (VCC), U14.91 (VCCint), U15.17 (Vcc), U15.29 (Vcc), U15.41 (Vcc), U15.9 (Vcc); no longer BT1.2 (-), C1.2, C4.2, C5.2, C6.1, C7.2, C8.2, C9.2, D4.1 (K), IC1.4 (GND), J2.19 (Pin_19), J2.2 (Pin_2), J2.22 (Pin_22), J2.24 (Pin_24), J2.26 (Pin_26), J2.28 (Pin_28), J2.30 (Pin_30), J2.40 (Pin_40), J3.1 (Pin_1), J3.11 (Pin_11), J3.13 (Pin_13), J3.15 (Pin_15), J3.17 (Pin_17), J3.19 (Pin_19), J3.21 (Pin_21), J3.23 (Pin_23), J3.25 (Pin_25), J3.27 (Pin_27), J3.29 (Pin_29), J3.3 (Pin_3), J3.31 (Pin_31), J3.33 (Pin_33), J3.5 (Pin_5), J3.7 (Pin_7), J3.9 (Pin_9), J4.3, J5.3, J7.10, J7.5, J7.6, J7.7, J7.8, JP1.2 (B), Q1.1 (E), R11.1, R12.1, R13.1, R29.2, R30.2, R44.1, R45.1, R48.2, R49.2, R50.2, R55.2, R6.1, RN2.1 (common), SW27.1, U1.1 (GND), U1.20 (GND), U11.12 (GND), U19.9 (GND), U2.12 (GND), U2.22 (SBA), U23.9 (GND), U24.12 (GND), U27.17 (WR2), U27.18 (VSS), U27.20 (RD2), U27.24 (~{ADS}), U28.12 (GND), U29.1 (~{OE}), U29.10 (GND), U3.10 (GND), U30.14 (GND), U31.16 (GND), U32.12 (GND), U34.12 (GND), U35.12 (GND), U36.1 (G1), U36.10 (GND), U36.8 (A6), U36.9 (A7), U37.8 (GND), U38.21 (CLK2), U38.22 (DRV), U38.31 (VSS), U4.8 (GND), U40.20 (GND), U40.7 (TL_EA), U44.1 (MOT), U44.12 (GND), U44.13 (~{CS}), U44.16 (GND), U46.10 (GND), U47.12 (GND), U48.12 (GND), U49.12 (GND), U50.16 (GND), U51.10 (GND), U52.1 (~{OE}), U52.10 (GND), U52.6 (4D), U52.7 (5D), U52.8 (6D), U52.9 (7D), U53.1 (~{OE}), U53.10 (GND), U54.1 (G1), U54.10 (GND), U54.19 (G2), U55.10 (GND), U56.14 (GND), U57.14 (GND), U57.16 (~{SP/EN}), U62.10 (P5), U62.11 (P6), U62.12 (P7), U62.14 (GND), U66.14 (GND), U66.2 (A12), U66.20 (~{CS}), U67.1 (SER), U67.6 (CLK_INH), U67.8 (GND), U68.1 (GND), U69.12 (GND), U71.1 (~{OE}), U71.10 (GND), U72.14 (GND), U72.20 (~{CS}), U73.12 (GND), U74.10 (GND), U75.10 (GND), U76.10 (GND), U77.10 (GND), U79.10 (GND), U80.10 (GND), U86.1 (G1), U86.10 (GND), U86.19 (G2), U87.10 (GND), Y1.4 (GND), Y2.4 (GND), Y3.4 (GND), Y5.4 (GND)
- net VD0: now also U14.37 (VD0)
- net VD1: now also U14.36 (VD1)
- net VD2: now also U14.35 (VD2)
- net VD3: now also U14.33 (VD3)
- net VD4: now also U14.32 (VD4)
- net VD5: now also U14.31 (VD5)
- net VD6: now also U14.30 (VD6)
- net VD7: now also U14.29 (VD7)
- net XD0: now also U47.11 (A7), U51.9 (A7); no longer U47.4 (A0), U51.2 (A0)
- net XD1: now also U47.10 (A6), U51.8 (A6); no longer U47.5 (A1), U51.3 (A1)
- net XD2: now also U47.9 (A5), U51.7 (A5); no longer U47.6 (A2), U51.4 (A2)
- net XD3: now also U47.8 (A4), U51.6 (A4); no longer U47.7 (A3), U51.5 (A3)
- net XD4: now also U47.7 (A3), U51.5 (A3); no longer U47.8 (A4), U51.6 (A4)
- net XD5: now also U47.6 (A2), U51.4 (A2); no longer U47.9 (A5), U51.7 (A5)
- net XD6: now also U47.5 (A1), U51.3 (A1); no longer U47.10 (A6), U51.8 (A6)
- net XD7: now also U47.4 (A0), U51.2 (A0); no longer U47.11 (A7), U51.9 (A7)
- net ~{ADOE}: now also U15.31 (~{ADOE})
- net ~{CBA}: now also U15.3 (CBA)
- net ~{CGA6845CS}: now also U69.16 (~{6845CS}); no longer U69.22 (~{6845CS})
- net ~{CGACOL}: now also U14.63 (~{CGACOL})
- net ~{CGAIO}: now also U69.23 (~{CGAIO}), U15.42 (~{CGAIO}); no longer U69.17 (~{CGAIO})
- net ~{CGAPALRD}: now also U69.15 (~{PALRD}); no longer U69.19 (~{PALRD})
- net ~{CGAPALWR}: now also U69.14 (~{PALWR}); no longer U69.18 (~{PALWR})
- net ~{CGARAM}: now also U15.23 (~{CGARAM})
- net ~{CGASTAT}: now also U69.22 (~{CGASTAT}), U14.57 (~{CGASTAT}); no longer U69.23 (~{CGASTAT})
- net ~{CG_OE}: now also U15.15 (~{CG_OE})
- net ~{CH}/AT: now also U14.79 (CH/~{AT})
- net ~{CLR_SR}: now also U14.45 (~{CLR_SR})
- net ~{Char Clk}: now also U14.80 (~{CHARCLK})
- net ~{FDCCS}: now also U48.10 (~{FDCCS})
- net ~{LOE}: no longer U46.19 (~{OE})
- net ~{MEMR}: now also U15.27 (~{MEMR})
- net ~{RDY}/WAIT: now also U15.22 (RDY/~{WAIT})
- net ~{VAOE}: now also U15.28 (~{VAOE})
- net ~{VROE}: now also U15.44 (~{VROE})
- net ~{VRWE}: now also U15.43 (~{VRWE})
- net 1.8432MHz: now reaches U27.14 (XIN), Y2.5 (OUTPUT)
- net ~{XDOE}: now reaches U11.19 (~{XDOE})
- net ~{XDOE}: now also U46.19 (~{OE})
- net +B/W renamed P4
- net P4: now also U14.100 (P4)
- net 25MHZ renamed 25MHz
- net 25MHz: now also U14.87 (GCLK1_25MHZ)
- net CGADIR renamed DT/R
- net DT/R: now also U46.1 (A->B), U47.3 (DIR), U51.1 (A->B)
- net HSync Dly renamed HSync
- net HSync: now also U14.94 (HSYNC)
- net UCBA renamed VSS
- net VSS: now also BT1.2 (-), C1.2, C4.2, C5.2, C6.1, C7.2, C8.2, C9.2, D4.1 (K), IC1.4 (GND), J2.19 (Pin_19), J2.2 (Pin_2), J2.22 (Pin_22), J2.24 (Pin_24), J2.26 (Pin_26), J2.28 (Pin_28), J2.30 (Pin_30), J2.40 (Pin_40), J3.1 (Pin_1), J3.11 (Pin_11), J3.13 (Pin_13), J3.15 (Pin_15), J3.17 (Pin_17), J3.19 (Pin_19), J3.21 (Pin_21), J3.23 (Pin_23), J3.25 (Pin_25), J3.27 (Pin_27), J3.29 (Pin_29), J3.3 (Pin_3), J3.31 (Pin_31), J3.33 (Pin_33), J3.5 (Pin_5), J3.7 (Pin_7), J3.9 (Pin_9), J4.3, J5.3, J7.10, J7.5, J7.6, J7.7, J7.8, JP1.2 (B), Q1.1 (E), R13.1, R29.2, R30.2, R44.1, R45.1, R48.2, R49.2, R50.2, R55.2, R6.1, RN2.1 (common), SW27.1, U1.1 (GND), U1.20 (GND), U11.12 (GND), U19.9 (GND), U2.12 (GND), U2.22 (SBA), U23.9 (GND), U24.12 (GND), U27.17 (WR2), U27.18 (VSS), U27.20 (RD2), U27.24 (~{ADS}), U28.12 (GND), U29.1 (~{OE}), U29.10 (GND), U3.10 (GND), U30.14 (GND), U31.16 (GND), U32.12 (GND), U34.12 (GND), U35.12 (GND), U36.1 (G1), U36.10 (GND), U36.8 (A6), U36.9 (A7), U37.8 (GND), U38.21 (CLK2), U38.22 (DRV), U38.31 (VSS), U4.8 (GND), U40.20 (GND), U40.7 (TL_EA), U44.1 (MOT), U44.12 (GND), U44.13 (~{CS}), U44.16 (GND), U46.10 (GND), U47.12 (GND), U48.12 (GND), U49.12 (GND), U50.16 (GND), U51.10 (GND), U52.1 (~{OE}), U52.10 (GND), U52.6 (4D), U52.7 (5D), U52.8 (6D), U52.9 (7D), U53.1 (~{OE}), U53.10 (GND), U54.1 (G1), U54.10 (GND), U54.19 (G2), U55.10 (GND), U56.14 (GND), U57.14 (GND), U57.16 (~{SP/EN}), U62.10 (P5), U62.11 (P6), U62.12 (P7), U62.14 (GND), U66.14 (GND), U66.2 (A12), U66.20 (~{CS}), U67.1 (SER), U67.6 (CLK_INH), U67.8 (GND), U68.1 (GND), U69.12 (GND), U71.1 (~{OE}), U71.10 (GND), U72.14 (GND), U72.20 (~{CS}), U73.12 (GND), U74.10 (GND), U75.10 (GND), U76.10 (GND), U77.10 (GND), U79.10 (GND), U80.10 (GND), U86.1 (G1), U86.10 (GND), U86.19 (G2), U87.10 (GND), Y1.4 (GND), Y2.4 (GND), Y3.4 (GND), Y5.4 (GND), J1.10 (GND), J1.2 (GND), U14.11 (GNDINT), U14.26 (GND), U14.38 (GND), U14.43 (GND), U14.59 (GND), U14.74 (GND), U14.86 (GND), U14.95 (GND), U15.16 (Gnd), U15.24 (Gnd), U15.36 (Gnd), U15.4 (Gnd)
- net VSync Dly renamed VSync
- net VSync: now also U14.92 (VSYNC)
- removed net XDIR: U46.1 (A->B), U47.3 (DIR), U48.14 (DIR), U51.1 (A->B)
- net ~{245CE} renamed ~{C245CE}
- net ~{C245CE}: now also U15.33 (~{C245CE})
- net ~{640BWOE} renamed ~{BW640OE}
- net ~{BW640OE}: now also U15.21 (~{BW640OE})
- net ~{646OE} renamed ~{C646OE}
- net ~{C646OE}: now also U15.5 (~{C646OE})
- net ~{CGACONT} renamed ~{CGACTL}
- net ~{CGACTL}: now also U14.61 (~{CGACTL})
- net ~{RESET} renamed  ~{RESET}
- net  ~{RESET}: now also U14.89 (GCLR_~{RESET}), U15.39 (GCLR)
- new net: J1.3 (TDO), R16.1, U15.32 (TDO)
- new net BW640: U14.48 (BW640), U15.18 (BW640)
- new net DotClk2: U14.41 (DOTCLK2), U67.7 (Clk)
- new net HS: U14.76 (HS), U68.39 (HS)
- new net Keyboard Data: C5.1, J5.1, R11.1, U40.27 (P10), U41.4
- new net Qc: U14.23 (Qc), U15.12 (Qc)
- new net TCK: J1.1 (TCK), U14.62 (TCK), U15.26 (TCK)
- new net TDI: J1.9 (TDI), R14.1, U14.4 (TDI)
- new net TDO/TDI: U14.73 (TDO), U15.1 (TDI)
- new net TMS: J1.5 (TMS), U14.15 (TMS), U15.7 (TMS)
- new net VS: U14.75 (VS), U68.40 (VS)
- no-connect marks 141 -> 139
Other:
- note added: "Character Generator EEPROM"
- note added: "Character ROM Select Each CGA Font 2K, VGA 4K 8K EEPROM Wide/Thin A11 - Thin selected"
- note added: "JTAG CPLD Programming Port Note TDI to Device 1, TDO to TDI then device 2 TDO to port"
- note added: "TODO ---- Finish pin mapping for 44 pin 1504 Configure 100 pin 1504 for Status Register Chip Labels for 44 & 100 pin chips Test Chips"
- note removed: "25.175MHz"
- note removed: "Attribute Latch"
- note removed: "Attribute Multiplexer PLD"
- note removed: "Blink Divider and HS VS"
- note removed: "CGA Colour Register"
- note removed: "CGA Control Register"
- note removed: "CGA Logic 1 PLD"
- note removed: "CGA Logic PLD 2"
- note removed: "CGA Status Register"
- note removed: "Character Gen. EEPROM"
- note removed: "Character ROM Select Each CGA Font 2K, VGA 4K 8K EEPROM"
- note removed: "Clock PLD"
- note removed: "Colour Multiplexer PLD"
- note removed: "First Flip Flop Syncs the CPUACT with the video Dot Clock so we don't have short DC Cycles from DCQ0-3"
- note removed: "Second Flip Flop delays the CPUACTSYNC by one video Dot Clock cycle otherwise we miss last Gated Dot Clock from CPUACTDCLK. CPUACTS1 ORed with CPUACTSYNC is used to gate the Dot Clock so it is extended."
- note removed: "TODO ---- Turbo logic for clock on 8284 - tbd Use 25.175MHz CLK - Yes should make CGA timing better PLD for 8288 bus controller, diagram in PPT - Done Remove wait state logic? No Needed for CGA and in PLD anyway - Done 16C550 Serial Port - Done 8255 PIA for Key Pad - Replaced by 74LS646 etc Done Update Monitor to use 16c550 and 74LS646 Debug monitor CONT and INT3 New keypad layout, reset and NMI?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"
- note removed: "Video Output PLD"
- moved on the sheet: C4, C5, C6, C7, C8, C9, J4, J5, R10, R11, R12, R9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
